File: Colorofon_V2_SMD.kicad_sch (KiCad schematic)
At the start: 94 parts, among them J1 Barrel_Jack_MountingPin, J2 AudioJack3, J3 691322310002, J4 691322310002, J5 691322310002, Q1 BC547, Q2 BC547, Q3 BC547, Q4 BD140, Q5 BD140, Q6 BD140, SW1 SW_Push, U1 LM358, U2 MCP6002-xP, U3 MCP6002-xP

Commit message: Change filters components
main clean board layout
Parts:
- removed Q4, Q5, Q6: BD140, Package_TO_SOT_THT:TO-126-3_Vertical, symbol Transistor_BJT:BD140
- removed R20, R22, R24: 100, Resistor_SMD:R_1206_3216Metric_Pad1.30x1.75mm_HandSolder, symbol Device:R
- removed SYM1: SYM_EasterEgg_42x60mm, Symbol:KiCad-Logo2_8mm_Copper, symbol Graphic:SYM_EasterEgg_42x60mm
- added C20: 100n, Capacitor_SMD:C_0805_2012Metric_Pad1.18x1.45mm_HandSolder, symbol Device:C
- added D7: LED, symbol Device:LED
- added Q4, Q5, Q6: PMV65XP, Package_TO_SOT_SMD:SOT-23_Handsoldering, symbol Transistor_FET:FDN340P
- added R28: 1,8k, Resistor_SMD:R_1206_3216Metric_Pad1.30x1.75mm_HandSolder, symbol Device:R
- added TP16: (no value), My_Library:PinHeader_1x02_P2.54mm_Vertical_Hand_Solder, symbol Connector:Conn_01x02_Pin
- C10, C11: value 22n -> 4,7n
- C12, C13: value 22n -> 680p
- C17, C18, C19: value 4.7u -> 10u
- H1, H2, H3, H4: footprint MountingHole:MountingHole_3.5mm_Pad_TopBottom -> MountingHole:MountingHole_2.2mm_M2_Pad_TopBottom
- R11: value 100k -> 1k
- R12: value 100k -> 560
- R13: value 510k -> 1M
- R14: value 510k -> 220k
- R15: value 510k -> 470k
- R7: value 100k -> 56k
- R8: value 100k -> 15k
- R9: value 100k -> 27k
- RV2, RV3: value 100k -> 200k
Connections:
- net +12V: now also Q4.2 (S), Q5.2 (S), Q6.2 (S), R28.2
- net GND: now also C20.1, D7.1 (K), TP16.2 (Pin_2)
- net at J3.1, R25.1: now also Q4.3 (D)
- net at R19.1: now also Q1.1 (C), Q4.1 (G)
- net at C6.2, RV1.2, RV2.3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: now also RV1.3; no longer RV1.1
- net at C6.1, R6.2, U2.2 (-): now also RV1.1; no longer RV1.3
- net at R21.1: now also Q2.1 (C), Q5.1 (G)
- net at J5.1, R27.1: now also Q6.3 (D)
- net at J4.1, R26.1: now also Q5.3 (D)
- net at Q3.1 (C): now also R23.1, Q6.1 (G)
- net at R1.1, R2.2, U1.3 (+): now also C20.2
- new net: D7.2 (A), R28.1, TP16.1 (Pin_1)
Other:
- note added: "1-4,1k +31dB"
- note added: "10-300Hz +31dB"
- note added: "5-20k +30dB"
- note added: "Zasilacz 800mA - 1 segment 14mA, 155mW"
- note added: "do poprawy"
- note added: "dodać przełącznik między 15k a 5k do basów i średnich?"
- note added: "doregulować tłumienie do potencjometrow"
- note added: "zmienic RV7 na res 5k"
- note removed: "1-4k +27dB"
- note removed: "20-300Hz +28dB"
- note removed: "5-18kHz 34dB"
- note removed: "sprawdzić 4,7 vs 10uF w połączeniu z trymerem 10k"
- note removed: "stworzyć symbol konektora wurtha"
- note removed: "ściągać STEP montażowych"
- title: (none) -> Colorofon V2
- moved on the sheet: C1, C2, C5, C7, H1, H2, H3, H4, R3, RV1, U1A, U1B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

Commit message: Update layout
Final layout for version 2
Parts:
- removed J2: AudioJack3, Connector_Audio:Jack_3.5mm_CUI_SJ-3523-SMT_Horizontal, symbol Connector_Audio:AudioJack3
- removed J3, J4, J5: 691322310002, My_Library:J_Wurth_WR-TBL_691322310002, symbol My_Symbols:691322310002
- removed Q1, Q2, Q3: BC547, My_Library:TO-92L_Wide_Hand, symbol Transistor_BJT:BC547
- removed R3: 0/10, Resistor_SMD:R_1206_3216Metric_Pad1.30x1.75mm_HandSolder, symbol Device:R
- removed RV1, RV4: 100k, My_Library:Potentiometer_Piher_T-16H_Single_Horizontal, symbol Device:R_Potentiometer
- removed RV2, RV3: 200k, My_Library:Potentiometer_Piher_T-16H_Single_Horizontal, symbol Device:R_Potentiometer
- removed RV5, RV6, RV7: 10k, My_Library:Potentiometer_Runtron_RM-065_Vertical_Hand_Solder, symbol Device:R_Potentiometer_Small
- removed SW1: SW_Push, Button_Switch_THT:SW_PUSH_1P1T_6x3.5mm_H4.3_APEM_MJTP1243, symbol Switch:SW_Push
- removed TP1, TP10, TP11, TP12, TP13, TP14, TP15, TP16, TP2, TP3, TP4, TP5, TP6, TP7, TP8, TP9: (no value), My_Library:PinHeader_1x02_P2.54mm_Vertical_Hand_Solder, symbol Connector:Conn_01x02_Pin
- added J2: AudioJack3_SwitchTR, My_Footprints:Jack_3.5mm_CUI_SJ2-3593D-SMT_Horizontal, symbol My_Symbols:AudioJack3_SwitchTR
- added J3, J4, J5: Connector 1x2 WE 691322310002, My_Footprints:J_Wurth_WR-TBL_691322310002, symbol My_Symbols:Connector 1x2 WE 691322310002
- added J6: Conn_01x02_Pin, My_Footprints:PinHeader_1x02_P2.54mm_Vertical_Hand_Solder, symbol Connector:Conn_01x02_Pin
- added Q1, Q2, Q3: BC847, Package_TO_SOT_SMD:SOT-23, symbol Transistor_BJT:BC847
- added R20, R30, R31, R32: 10, Resistor_SMD:R_1206_3216Metric_Pad1.30x1.75mm_HandSolder, symbol Device:R
- added R22, R24, R29: 1k, Resistor_SMD:R_1206_3216Metric_Pad1.30x1.75mm_HandSolder, symbol Device:R
- added RV1: 100k, My_Footprints:Potentiometer_Piher_T-16H_Single_Horizontal, symbol My_Symbols:R_Potentiometer
- added RV2, RV3, RV4: 1k, My_Footprints:Potentiometer_Piher_T-16H_Single_Horizontal, symbol My_Symbols:R_Potentiometer
- added RV5, RV6, RV7: 10k, My_Footprints:Potentiometer_Runtron_RM-065_Vertical_Hand_Solder, symbol My_Symbols:R_Potentiometer_Small
- added SW2: SW_SPDT, My_Footprints:SW_Toggle_Blue_wSlots, symbol Switch:SW_SPDT
- C10: value 4,7n -> 680p
- C11: value 4,7n -> 1n
- C12: value 680p -> 100p
- C13: value 680p -> 4,7n
- C14, C15, C16, C4, C6: now fitted; now in the parts list
- C8: value 22n -> 10n
- C9: value 22n -> 33n
- H1, H2, H3, H4: footprint MountingHole:MountingHole_2.2mm_M2_Pad_TopBottom -> MountingHole:MountingHole_2.2mm_M2
- J1: footprint My_Library:BarrelJack_Horizontal -> My_Footprints:BarrelJack_Horizontal
- Q4, Q5, Q6: footprint Package_TO_SOT_SMD:SOT-23_Handsoldering -> Package_TO_SOT_SMD:SOT-23
- R11: value 1k -> 10k
- R13: value 1M -> 560k
- R14: value 220k -> 660k
- R4, R5, R6: value 5.1k -> 5,1k
- R7: value 56k -> 1k
- R8: value 15k -> 1k
- R9: value 27k -> 1k
- U2, U3: value MCP6002-xP -> LM358
Connections:
- net +12V: now also SW2.3 (C)
- net GND: now also U1.5 (+), U1.6 (-), J2.S, J3.2, J4.2, J5.2, J6.2 (Pin_2)
- net Vref: now also Q1.2 (E), Q2.2 (E), Q3.2 (E), R22.2, R24.2, R29.2, R32.2, RV2.1, RV3.1, RV4.1, RV5.1, RV5.2, RV6.1, RV6.2, RV7.1, RV7.2
- net at R9.1: now also RV4.2
- net at C10.1, R14.2, U3.1: now also R24.1, R30.1; no longer D2.2 (A)
- net at C6.1, R6.2, U2.2 (-): now also RV1.1
- net at C6.2, U2.1: now also RV1.2, RV1.3, RV2.3, RV3.3, RV4.3
- net at Q5.1 (G), R21.1: now also Q2.3 (C)
- net at Q4.1 (G), R19.1: now also Q1.3 (C)
- net at R7.1: now also RV2.2
- net at R4.1: now also J2.T, J2.TN
- net at C8.1, R13.2, U2.7: now also R20.1, R29.1; no longer D1.2 (A)
- net at Q6.3 (D), R27.1: now also J5.1
- net at Q5.3 (D), R26.1: now also J4.1
- net at R5.1: now also J2.R, J2.RN
- net at R16.2: now also Q1.1 (B)
- net at C19.2, D3.1 (K), R18.1: now also RV7.3
- net at C12.1, R15.2, U3.7: now also R22.1, R31.1; no longer D3.2 (A)
- net at C17.2, D1.1 (K), R16.1: now also RV5.3
- net at R8.1: now also RV3.2
- net at R17.2: now also Q2.1 (B)
- net at C18.2, D2.1 (K), R17.1: now also RV6.3
- net at Q6.1 (G), R23.1: now also Q3.3 (C)
- net at R18.2: now also Q3.1 (B)
- net at D7.2 (A), R28.1: now also J6.1 (Pin_1)
- net at Q4.3 (D), R25.1: now also J3.1
- net at U1.1, U1.2 (-): now also R32.1
- net at J1.1: now also SW2.2 (B)
- new net: D2.2 (A), R30.2
- new net: D3.2 (A), R31.2
- new net: D1.2 (A), R20.2
- no-connect marks 3 -> 2
Other:
- note added: "10-400Hz +30dB"
- note removed: "10-300Hz +31dB"
- note removed: "do poprawy"
- note removed: "doregulować tłumienie do potencjometrow"
- note removed: "zmienic RV7 na res 5k"
- moved on the sheet: C1, C17, C18, C19, C2, D1, D2, D3, D4, D5, D6, D7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
